File: Kicad_PCB_Files/leds.sch (KiCad schematic (older format))
At the start: 13 parts, among them U3 74LS04

Commit message: Add files via upload
Parts:
- R3, R4, R5, R6, R7, R8, U3: Vendor (none) -> ETSG
Changed lines of the file:
@@
 F 2 "Package_DIP:DIP-14_W7.62mm_LongPads" H 5800 5600 50  0001 C CNN
 F 3 "http://www.ti.com/lit/gpn/sn74LS04" H 5800 5600 50  0001 C CNN
+F 4 "ETSG" H 5800 5600 50  0001 C CNN "Vendor"
 	7    5800 5600
 	1    0    0    -1
@@
 F 2 "Resistor_SMD:R_0805_2012Metric_Pad1.15x1.40mm_HandSolder" V 3680 1500 50  0001 C CNN
 F 3 "~" H 3750 1500 50  0001 C CNN
+F 4 "ETSG" V 3750 1500 50  0001 C CNN "Vendor"
 	1    3750 1500
 	0    1    1    0
@@
 F 2 "Resistor_SMD:R_0805_2012Metric_Pad1.15x1.40mm_HandSolder" V 3680 2000 50  0001 C CNN
 F 3 "~" H 3750 2000 50  0001 C CNN
+F 4 "ETSG" V 3750 2000 50  0001 C CNN "Vendor"
 	1    3750 2000
 	0    1    1    0
@@
 F 2 "Resistor_SMD:R_0805_2012Metric_Pad1.15x1.40mm_HandSolder" V 3680 2500 50  0001 C CNN
 F 3 "~" H 3750 2500 50  0001 C CNN
+F 4 "ETSG" V 3750 2500 50  0001 C CNN "Vendor"
 	1    3750 2500
 	0    1    1    0
@@
 F 2 "Resistor_SMD:R_0805_2012Metric_Pad1.15x1.40mm_HandSolder" V 3680 3000 50  0001 C CNN
 F 3 "~" H 3750 3000 50  0001 C CNN
+F 4 "ETSG" V 3750 3000 50  0001 C CNN "Vendor"
 	1    3750 3000
 	0    1    1    0
@@
 F 2 "Resistor_SMD:R_0805_2012Metric_Pad1.15x1.40mm_HandSolder" V 3680 3500 50  0001 C CNN
 F 3 "~" H 3750 3500 50  0001 C CNN
+F 4 "ETSG" V 3750 3500 50  0001 C CNN "Vendor"
 	1    3750 3500
 	0    1    1    0
@@
 F 2 "Resistor_SMD:R_0805_2012Metric_Pad1.15x1.40mm_HandSolder" V 3680 3950 50  0001 C CNN
 F 3 "~" H 3750 3950 50  0001 C CNN
+F 4 "ETSG" V 3750 3950 50  0001 C CNN "Vendor"
 	1    3750 3950
 	0    1    1    0

Commit message: Add files via upload
Parts:
- D5, D6, GPS_RX1, LORA_SEND1, NETWORK_JOIN1, SIGNAL_STR1: footprint LED_THT:LED_D3.0mm -> LED_SMD:LED_0805_2012Metric_Pad1.15x1.40mm_HandSolder
Changed lines of the file:
@@
 F 0 "LORA_SEND1" H 5843 1245 50  0000 C CNN
 F 1 "LED" H 5843 1336 50  0000 C CNN
-F 2 "LED_THT:LED_D3.0mm" H 5850 1500 50  0001 C CNN
+F 2 "LED_SMD:LED_0805_2012Metric_Pad1.15x1.40mm_HandSolder" H 5850 1500 50  0001 C CNN
 F 3 "~" H 5850 1500 50  0001 C CNN
 	1    5850 1500
@@
 F 0 "GPS_RX1" H 5843 1745 50  0000 C CNN
 F 1 "LED" H 5843 1836 50  0000 C CNN
-F 2 "LED_THT:LED_D3.0mm" H 5850 2000 50  0001 C CNN
+F 2 "LED_SMD:LED_0805_2012Metric_Pad1.15x1.40mm_HandSolder" H 5850 2000 50  0001 C CNN
 F 3 "~" H 5850 2000 50  0001 C CNN
 	1    5850 2000
@@
 F 0 "NETWORK_JOIN1" H 5843 2245 50  0000 C CNN
 F 1 "LED" H 5843 2336 50  0000 C CNN
-F 2 "LED_THT:LED_D3.0mm" H 5850 2500 50  0001 C CNN
+F 2 "LED_SMD:LED_0805_2012Metric_Pad1.15x1.40mm_HandSolder" H 5850 2500 50  0001 C CNN
 F 3 "~" H 5850 2500 50  0001 C CNN
 	1    5850 2500
@@
 F 0 "SIGNAL_STR1" H 5843 2745 50  0000 C CNN
 F 1 "LED" H 5843 2836 50  0000 C CNN
-F 2 "LED_THT:LED_D3.0mm" H 5850 3000 50  0001 C CNN
+F 2 "LED_SMD:LED_0805_2012Metric_Pad1.15x1.40mm_HandSolder" H 5850 3000 50  0001 C CNN
 F 3 "~" H 5850 3000 50  0001 C CNN
 	1    5850 3000
@@
 F 0 "D5" H 5843 3245 50  0000 C CNN
 F 1 "LED" H 5843 3336 50  0000 C CNN
-F 2 "LED_THT:LED_D3.0mm" H 5850 3500 50  0001 C CNN
+F 2 "LED_SMD:LED_0805_2012Metric_Pad1.15x1.40mm_HandSolder" H 5850 3500 50  0001 C CNN
 F 3 "~" H 5850 3500 50  0001 C CNN
 	1    5850 3500
@@
 F 0 "D6" H 5843 3695 50  0000 C CNN
 F 1 "LED" H 5843 3786 50  0000 C CNN
-F 2 "LED_THT:LED_D3.0mm" H 5850 3950 50  0001 C CNN
+F 2 "LED_SMD:LED_0805_2012Metric_Pad1.15x1.40mm_HandSolder" H 5850 3950 50  0001 C CNN
 F 3 "~" H 5850 3950 50  0001 C CNN
 	1    5850 3950
