File: Kicad_PCB_Files/BarGraph/BarGraph.kicad_pcb (KiCad board)
At the start: 2 copper layers, 30.5 x 98.9 mm, 12 parts, among them J1 USB_B_Micro

Commit message: Add files via upload
Parts:
- removed 5V, SIGNAL: TestPoint, TestPoint:TestPoint_Pad_2.5x2.5mm
- removed BRIGHTNESS CONTROL: 100k, Potentiometer_THT:Potentiometer_Alps_RK09K_Single_Horizontal
- removed C1 22U: 22u, Capacitor_SMD:C_0603_1608Metric_Pad1.05x0.95mm_HandSolder
- removed LED BAR GRAPH: LED-Bar-Graph, ledbar:led-bar-graph-10
- removed LED DRIVER: LM3914VX_NOPB, Package_LCC:PLCC-20
- removed R1 10K: 10k, Resistor_SMD:R_0603_1608Metric_Pad1.05x0.95mm_HandSolder
- removed R2 OPT 1K6: 1.6k, Resistor_SMD:R_0603_1608Metric_Pad1.05x0.95mm_HandSolder
- removed R3 OPT 3K6: 3.6k, Resistor_SMD:R_0603_1608Metric_Pad1.05x0.95mm_HandSolder
- removed R4 1K6: 1.6k, Resistor_SMD:R_0603_1608Metric_Pad1.05x0.95mm_HandSolder
- removed REF OUT: TestPoint, TestPoint:TestPoint_Pad_2.5x2.5mm
- added C1: 22u, Capacitor_THT:CP_Radial_D5.0mm_P2.50mm, F.Cu at (142.2, 116.8)
- added H1: MountingHole, MountingHole:MountingHole_4mm_Pad, F.Cu at (143.0, 41.0)
- added H2: MountingHole, MountingHole:MountingHole_4mm_Pad, F.Cu at (162.0, 41.0)
- added H3: MountingHole, MountingHole:MountingHole_4mm_Pad, F.Cu at (162.0, 89.0)
- added H4: MountingHole, MountingHole:MountingHole_4mm_Pad, F.Cu at (162.0, 118.2)
- added R1: 10k, Resistor_THT:R_Axial_DIN0207_L6.3mm_D2.5mm_P10.16mm_Horizontal, F.Cu at (141.0, 121.9)
- added R2: 1.6k, Resistor_THT:R_Axial_DIN0207_L6.3mm_D2.5mm_P2.54mm_Vertical, F.Cu at (165.1, 130.8)
- added R3: 3.6k, Resistor_THT:R_Axial_DIN0207_L6.3mm_D2.5mm_P2.54mm_Vertical, F.Cu at (165.1, 127.0)
- added R4: 1.6k, Resistor_THT:R_Axial_DIN0207_L6.3mm_D2.5mm_P10.16mm_Horizontal, F.Cu at (157.5, 113.0)
- added TP1: TestPoint, TestPoint:TestPoint_Pad_2.5x2.5mm, F.Cu at (147.6, 113.8)
- added TP2: TestPoint, TestPoint:TestPoint_Pad_2.5x2.5mm, F.Cu at (147.1, 121.4)
- added TP4: TestPoint, TestPoint:TestPoint_Pad_2.5x2.5mm, F.Cu at (164.7, 80.5)
- added U1: LED-Bar-Graph, ledbar:led-bar-graph-10, F.Cu at (152.4, 72.4)
- added U2: LM3914N, Package_DIP:DIP-18_W7.62mm_Socket_LongPads, F.Cu at (142.2, 109.2)
- J1: value USB_B_Micro -> USB_B; footprint Connector_USB:USB_Micro-B_Amphenol_10103594-0001LF_Horizontal -> SmartGluttonV1:USB_B_Molex_USB-67068-xx1x_StraightTab_Horizontal
- moved J1 4.83 mm to (153.7, 127.0), turned to 270 degrees
Connections:
- J1 pad 4: Net-(J1-Pad4) -> GND
Routing:
- net Net-(U1-Pad1): track 0.00 -> 75.6 mm
- net Net-(IC1-Pad12): track 67.8 -> 0.00 mm
- net Net-(U1-Pad2): track 0.00 -> 61.0 mm
- net Net-(IC1-Pad13): track 59.4 -> 0.00 mm
- net Net-(U1-Pad3): track 0.00 -> 52.7 mm
- net Net-(IC1-Pad14): track 52.6 -> 0.00 mm
- net Net-(IC1-Pad15): track 46.6 -> 0.00 mm
- net Net-(U1-Pad4): track 0.00 -> 44.8 mm
- net Net-(IC1-Pad16): track 41.5 -> 0.00 mm
- net Net-(U1-Pad5): track 0.00 -> 38.4 mm
- net Net-(IC1-Pad17): track 36.1 -> 0.00 mm
- net Net-(U1-Pad6): track 0.00 -> 33.0 mm
- net Net-(IC1-Pad18): track 30.6 -> 0.00 mm
- net GND: track 33.5 -> 3.05 mm, vias 3 -> 1
- net Net-(IC1-Pad19): track 29.0 -> 0.00 mm
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Other:
- net class Default: trace_width 0.25 -> 0.35
- board text added: "10K"
- board text added: "1K6"
- board text added: "22U"
- board text added: "5V"
- board text added: "GND"
- board text added: "OPT"
- board text added: "SIG"

Commit message: Add files via upload
Parts:
- moved H4 32.0 mm to (140.0, 95.0)
- moved H2 23.4 mm to (140.0, 49.0)
- moved H1 18.8 mm to (160.0, 49.0)
- moved R1 11.4 mm to (152.0, 119.0)
- moved C1 11.2 mm to (146.5, 127.2)
- moved R3 9.18 mm to (160.2, 119.2), turned to 270 degrees
- moved TP4 7.50 mm to (157.8, 77.8)
- moved R2 7.38 mm to (160.2, 125.2), turned to 270 degrees
- moved TP2 7.21 mm to (140.0, 120.0)
- moved J1 6.47 mm to (151.2, 133.0)
- moved TP1 6.35 mm to (146.2, 120.0)
- moved H3 6.32 mm to (160.0, 95.0)
- moved R4 6.15 mm to (156.0, 119.0)
- moved U2 5.19 mm to (140.2, 114.0)
- moved U1 4.72 mm to (150.0, 76.5)
Routing:
- net GND: track 3.05 -> 8.91 mm, vias 1 -> 0
- net Net-(U1-Pad7): track 27.6 -> 31.8 mm
- net Net-(U1-Pad8): track 22.9 -> 26.8 mm
- net Net-(U1-Pad9): track 18.5 -> 20.7 mm
- net Net-(R4-Pad1): track 3.81 -> 5.22 mm
- net Net-(U1-Pad10): track 13.2 -> 14.5 mm
- net Net-(J1-Pad3): track 11.5 -> 10.3 mm
- net Net-(U1-Pad3): track 52.7 -> 53.3 mm
- net Net-(U1-Pad1): track 75.6 -> 76.2 mm
- net Net-(C1-Pad1): track 19.8 -> 19.2 mm
- net Net-(U1-Pad4): track 44.8 -> 45.3 mm
Other:
- board size 30.5 x 98.9 mm -> 30 x 100 mm
- net class Default: clearance 0.2 -> 0.3
- net class Power: clearance 0.2 -> 0.3
- rule trace_clearance: 0.2 -> 0.3
- board text added: "LED BAR GRAPH 1.2"
- board text removed: "5V"
- board text removed: "OPT"
- board text removed: "PIN 1"

Commit message: Add files via upload
Parts:
- added R5: 10k, Resistor_THT:R_Axial_DIN0207_L6.3mm_D2.5mm_P10.16mm_Horizontal, F.Cu at (155.5, 119.0)
- H1, H2, H3, H4: footprint MountingHole:MountingHole_4mm_Pad -> MountingHole:MountingHole_4mm
- moved TP4 3.25 mm to (161.0, 77.8)
- moved R2 2.80 mm to (163.0, 124.8)
- moved R3 2.80 mm to (163.0, 118.7)
- moved R4 2.50 mm to (158.5, 119.0)
- moved U1 0.46 mm to (150.0, 76.0)
Connections:
- R2 pad 1: Net-(J1-Pad2) -> Net-(R2-Pad1)
- R3 pad 2: Net-(J1-Pad2) -> Net-(R2-Pad1)
- U2 pad 6: Net-(J1-Pad2) -> Net-(R2-Pad1)
Routing:
- net Net-(U1-Pad1): track 76.2 -> 23.8 mm
- net Net-(U1-Pad10): track 14.5 -> 66.2 mm
- net Net-(U1-Pad9): track 20.7 -> 59.2 mm
- net Net-(U1-Pad2): track 61.5 -> 27.2 mm
- net Net-(J1-Pad2): track 37.6 -> 8.34 mm
- net Net-(U1-Pad8): track 26.8 -> 52.1 mm
- net Net-(U1-Pad3): track 53.3 -> 30.9 mm
- net Net-(R2-Pad1): track 0.00 -> 19.0 mm
- net Net-(U1-Pad7): track 31.8 -> 45.0 mm
- net Net-(U1-Pad6): track 32.8 -> 45.3 mm
- net Net-(U1-Pad4): track 45.3 -> 36.6 mm
- net Net-(U1-Pad5): track 38.3 -> 40.7 mm
- net Net-(R4-Pad1): track 5.22 -> 6.26 mm
Other:
- board text added: "5V"
- board text added: "LED BAR GRAPH 1.3"
- board text removed: "LED BAR GRAPH 1.2"
